File: usb-base.kicad_pcb (KiCad board)
At the start: 4 copper layers, 100 x 100 mm, 19 parts, among them J1 USB3_B, U1 CYUSB3082-FCAXI, U2 TPS25221, U3 TPS62161DSG, U4 LFE5U-25F-6BG256C, U5 TPS62160DSG, U6 TPS62162DSG, Y1 24MHz, Y2 25MHz

Commit message: lots of work on layout
Parts:
- removed J1: USB3_B, Infineon:SAMTEC_USB3-B-S-F-TH
- removed Y2: 25MHz, Crystal:Crystal_SMD_SeikoEpson_TSX3225-4Pin_3.2x2.5mm
- added C12: 100n, Capacitor_SMD:C_0402_1005Metric, F.Cu at (114.5, 56.9)
- added C13: 100n, Capacitor_SMD:C_0402_1005Metric, F.Cu at (114.5, 57.9)
- added C14: 10u, Capacitor_SMD:C_0805_2012Metric, F.Cu at (116.8, 87.5)
- added C15: 22u, Capacitor_SMD:C_1206_3216Metric, F.Cu at (112.8, 92.2)
- added C7: 100n, Capacitor_SMD:C_0402_1005Metric, F.Cu at (114.5, 52.7)
- added C8: 100n, Capacitor_SMD:C_0402_1005Metric, F.Cu at (114.5, 51.8)
- added J2: USB_C_Receptacle, Connector_USB:USB_C_Receptacle_Amphenol_12401548E4-2A, F.Cu at (107.5, 54.2)
- added L4: 2.2u, Inductor_SMD:L_Sunlord_SWPA3015S, F.Cu at (112.3, 88.3)
- added R4: 20k, Resistor_SMD:R_0402_1005Metric, F.Cu at (97.8, 99.7)
- added R5: 7.5k, Resistor_SMD:R_0402_1005Metric, F.Cu at (97.8, 101.7)
- added R6: R, Resistor_SMD:R_0402_1005Metric, F.Cu at (114.8, 97.5)
- added R7: R, Resistor_SMD:R_0402_1005Metric, F.Cu at (114.8, 99.5)
- added R8: R, Resistor_SMD:R_0402_1005Metric, F.Cu at (114.5, 58.9)
- added R9: R, Resistor_SMD:R_0402_1005Metric, F.Cu at (114.5, 53.7)
- added U7: Si5340, Package_DFN_QFN:QFN-44-1EP_7x7mm_P0.5mm_EP5.2x5.2mm, F.Cu at (140.6, 46.5)
- added U8: TPS62160DSG, Package_SON:WSON-8-1EP_2x2mm_P0.5mm_EP0.9x1.6mm_ThermalVias, F.Cu at (117.8, 92.5)
- U1: footprint Infineon:BGA169N075P13X13_10X10X120 -> library:BGA169N075P13X13_10X10X120
- moved U2 86.3 mm to (99.2, 32.9)
- moved C9 76.5 mm to (99.2, 36.9)
- moved C11 69.5 mm to (100.0, 83.8)
- moved C10 66.7 mm to (95.7, 89.1)
- moved L3 65.6 mm to (100.3, 89.2)
- moved U5 65.6 mm to (100.2, 93.3)
- moved C1 57.8 mm to (80.1, 86.3)
- moved U3 57.8 mm to (84.5, 86.7)
- moved L2 57.8 mm to (75.5, 91.7)
- moved C2 57.1 mm to (82.0, 92.4)
- moved C5 16.9 mm to (133.2, 93.6)
- moved L1 12.8 mm to (137.3, 86.4)
- moved C6 11.3 mm to (133.3, 89.7)
- moved U6 11.3 mm to (137.7, 90.8)
- moved U4 5.30 mm to (139.4, 59.2)
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Connections:
- net +1V8 renamed +1.8V
- net +2V5 renamed +2.5V
- net 24MHz renamed 24MHZ
- U1 pad A3: +3V3 -> +3.3V
- U1 pad C11: +3V3 -> +3.3V
- U1 pad C3: +3V3 -> +3.3V
- U1 pad C5: +3V3 -> +3.3V
- U1 pad C7: +3V3 -> +3.3V
- U1 pad C9: +3V3 -> +3.3V
- U1 pad E3: +3V3 -> +3.3V
- U1 pad E5: unconnected-(U1C-P7_2_SPIDAT2-PadE5) -> CLK_SPI_MOSI
- U1 pad E6: unconnected-(U1C-P7_3_SPIDAT3-PadE6) -> CLK_SPI_MISO
- U1 pad F5: unconnected-(U1C-P7_0_SPIDAT0-PadF5) -> CLK_SPI_CLK
- U1 pad F6: unconnected-(U1C-P7_1_SPIDAT1-PadF6) -> CLK_SPI_CS
- U1 pad F7: +3V3 -> +3.3V
- U1 pad G3: +3V3 -> +3.3V
- U1 pad J3: +3V3 -> +3.3V
- U1 pad L10: +3V3 -> +3.3V
- U1 pad L13: +3V3 -> +3.3V
- U1 pad M12: +3V3 -> +3.3V
- U1 pad M3: USBSS_RX+ -> USBSS_RX1+
- U1 pad M5: USBSS_TX+ -> USBSS_TX1+
- U1 pad M7: unconnected-(U1B-USB3TX2_P-PadM7) -> USBSS_RX2+
- U1 pad M9: unconnected-(U1B-USB3RX2_P-PadM9) -> USBSS_TX2+
- U1 pad N3: USBSS_RX- -> USBSS_RX1-
- U1 pad N5: USBSS_TX- -> USBSS_TX1-
- U1 pad N7: unconnected-(U1B-USB3TX2_N-PadN7) -> USBSS_RX2-
- U1 pad N9: unconnected-(U1B-USB3RX2_N-PadN9) -> USBSS_TX2-
- U4 pad A7: 25MHz -> 100MHZ
- U4 pad C8: unconnected-(U4C-PT44A/+/PCLKT1_0-PadC8) -> CLK2
- U4 pad E8: unconnected-(U4C-PT42A/+/PCLKT1_1-PadE8) -> CLK1
- U4 pad F10: +3V3 -> +3.3V
- U4 pad F11: +3V3 -> +3.3V
- U4 pad F6: +3V3 -> +3.3V
- U4 pad F7: +3V3 -> +3.3V
- U4 pad H11: +3V3 -> +3.3V
- U4 pad H6: +3V3 -> +3.3V
- U4 pad H7: +3V3 -> +3.3V
- U4 pad J11: +3V3 -> +3.3V
- U4 pad J6: +3V3 -> +3.3V
- U4 pad J7: +3V3 -> +3.3V
- U4 pad K11: +3V3 -> +3.3V
- U4 pad L11: +3V3 -> +3.3V
- U4 pad L6: +3V3 -> +3.3V
- U4 pad N10: +3V3 -> +3.3V
Routing:
- net CLK_SPI_MISO: track 0.00 -> 26.8 mm, vias 0 -> 2
- net CLK_SPI_MOSI: track 0.00 -> 25.8 mm, vias 0 -> 2
- net CLK_SPI_CS: track 0.00 -> 25.0 mm, vias 0 -> 2
- net CLK_SPI_CLK: track 0.00 -> 24.0 mm, vias 0 -> 2
- net USBHS_D-: track 0.00 -> 18.6 mm
- net USBHS_D+: track 0.00 -> 17.8 mm, vias 0 -> 1
- net USBSS_RX1+: track 0.00 -> 15.2 mm, vias 0 -> 1
- net USBSS_RX1-: track 0.00 -> 14.7 mm, vias 0 -> 1
- net +3V3: track 13.8 -> 0.00 mm, vias 17 -> 0
- net +3.3V: track 5.60 -> 17.5 mm, vias 2 -> 20
- net P0D14: track 10.7 -> 0.10 mm
- net 100MHZ: track 0.00 -> 9.96 mm
- net Net-(J2-CC2): track 0.00 -> 9.54 mm, vias 0 -> 1
- net USBSS_TX1+: track 0.00 -> 9.15 mm
- net CLK1: track 0.00 -> 8.80 mm
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- added copper zone on B.Cu, net GND
- added copper zone on In2.Cu, net GND
Other:
- board size 100 x 100 mm -> 50 x 35 mm
- board text added: "24 MHz"
- board text added: "ECP5"
- board text added: "FX5"
- board text added: "Si5340"
- board text added: "USB 3.2"

Commit message: Lots of routing for connectors
Parts:
- removed U7: Si5340, Package_DFN_QFN:QFN-44-1EP_7x7mm_P0.5mm_EP5.2x5.2mm
- added J1: Conn_02x35_Odd_Even, Connector_Hirose_DF40:Hirose_DF40C-70DS-0.4V_2x35_P0.4mm, F.Cu at (144.8, 51.0)
- added J2: Conn_02x35_Odd_Even, Connector_Hirose_DF40:Hirose_DF40C-70DS-0.4V_2x35_P0.4mm, F.Cu at (144.8, 95.0)
- added Y2: 50MHz, Crystal:Crystal_SMD_SeikoEpson_TSX3225-4Pin_3.2x2.5mm, F.Cu at (136.6, 61.6)
- J3: renamed from J2; footprint Connector_USB:USB_C_Receptacle_Amphenol_12401548E4-2A -> Connector_USB:USB_C_Receptacle_Amphenol_12401610E4-2A
- moved L2 55.0 mm to (130.4, 89.9)
- moved C2 53.4 mm to (135.4, 90.1)
- moved C1 50.1 mm to (130.2, 86.3)
- moved U3 50.1 mm to (134.7, 86.7)
- moved C6 40.2 mm to (120.9, 51.5)
- moved C5 40.2 mm to (120.8, 55.4)
- moved L1 37.1 mm to (125.4, 51.3)
- moved U6 37.1 mm to (125.8, 55.6)
- moved U2 20.0 mm to (109.3, 50.2)
- moved C9 19.2 mm to (109.3, 53.2), turned to 180 degrees
- moved R5 16.2 mm to (112.3, 94.5)
- moved L3 13.6 mm to (113.8, 87.5)
- moved C10 13.6 mm to (109.2, 87.4)
- moved U5 13.6 mm to (113.7, 91.7)
- moved U1 12.6 mm to (122.0, 71.7)
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Connections:
- net PMODE renamed /PMODE
- U1 pad H13: DONE -> GPIO_1
- U1 pad J12: GPIO_1 -> DONE
- U1 pad K6: unconnected-(U1B-XRES_N-PadK6) -> /RESET
- U4 pad A7: 100MHZ -> 50MHz
- U4 pad B15: D0_1 -> D0_8
- U4 pad B16: D0_0 -> D0_10
- U4 pad C14: D0_2 -> D0_4
- U4 pad C15: D0_5 -> D0_12
- U4 pad C16: D0_4 -> D0_14
- U4 pad C8: CLK2 -> unconnected-(U4C-PT44A/+/PCLKT1_0-PadC8)
- U4 pad D14: D0_3 -> D0_6
- U4 pad D16: D0_8 -> D0_16
- U4 pad E14: D0_6 -> D0_11
- U4 pad E15: D0_9 -> D0_18
- U4 pad E16: D0_13 -> D0_20
- U4 pad E8: CLK1 -> unconnected-(U4C-PT42A/+/PCLKT1_1-PadE8)
- U4 pad F12: unconnected-(U4D-PR17D/-/RDQ17-PadF12) -> D0_0
- U4 pad F13: D0_10 -> D0_2
- U4 pad F14: D0_7 -> D0_15
- U4 pad F15: D0_12 -> D0_22
- U4 pad F16: D0_14 -> D0_24
- U4 pad G12: unconnected-(U4D-PR20A/+/HS/RDQ17-PadG12) -> D0_3
- U4 pad G13: D0_11 -> D0_7
- U4 pad G14: D0_16 -> D0_17
- U4 pad G15: D0_15 -> D0_25
- U4 pad G16: D0_20 -> D0_26
- U4 pad H12: unconnected-(U4D-PR26A/+/HS/RDQ29-PadH12) -> D0_1
- U4 pad H13: D0_18 -> D0_13
- U4 pad H14: D0_17 -> D0_19
- U4 pad H15: D0_21 -> D0_27
- U4 pad J12: unconnected-(U4D-PR26D/-/RDQ29-PadJ12) -> D0_5
- U4 pad J13: D0_19 -> D0_9
- U4 pad J14: D0_22 -> D0_21
- U4 pad J15: D0_25 -> D0_28
- U4 pad J16: D0_24 -> D0_29
- U4 pad K12: D1_5 -> D1_30
- U4 pad K13: D1_4 -> D1_28
- U4 pad K15: D0_27 -> D0_30
- U4 pad K16: D0_26 -> D0_31
- U4 pad L12: D1_7 -> D1_6
- U4 pad L13: D1_6 -> D1_26
- U4 pad L14: D1_10 -> D1_24
- U4 pad L15: D1_1 -> D1_31
- U4 pad L16: D1_0 -> D1_29
- U4 pad M10: unconnected-(U4I-TDO-PadM10) -> TDO
- U4 pad M11: unconnected-(U4E-PR68A/+/HS/RDQ65-PadM11) -> D1_2
- U4 pad M12: D1_25 -> D1_4
- U4 pad M13: D1_14 -> D1_20
- U4 pad M14: D1_11 -> D1_22
- U4 pad M15: D1_3 -> D1_27
- U4 pad M16: D1_2 -> D1_25
- U4 pad M7: GPIO_5 -> GPIO_2
- U4 pad N11: unconnected-(U4E-PR68B/-/HS/RDQ65-PadN11) -> D1_0
- U4 pad N12: D1_26 -> D1_10
- U4 pad N13: D1_16 -> D1_14
- U4 pad N14: D1_15 -> D1_18
- U4 pad N16: D1_8 -> D1_23
- U4 pad N7: GPIO_2 -> unconnected-(U4H-PB9A/+/D3/IO3-PadN7)
- U4 pad P11: unconnected-(U4E-PR68C/+/LRC_GPLL0T_IN/RDQ65-PadP11) -> D1_1
- U4 pad P12: D1_27 -> D1_8
- U4 pad P13: D1_20 -> D1_12
- U4 pad P14: D1_17 -> D1_16
- U4 pad P15: D1_9 -> D1_19
- U4 pad P16: D1_12 -> D1_21
- U4 pad P7: GPIO_3 -> GPIO_4
- U4 pad R11: unconnected-(U4I-TDI-PadR11) -> TDI
- U4 pad R12: D1_24 -> D1_3
- U4 pad R13: D1_22 -> D1_7
- U4 pad R14: D1_21 -> D1_11
- U4 pad R15: D1_18 -> D1_15
- U4 pad R16: D1_13 -> D1_17
- U4 pad R6: GPIO_0 -> GPIO_5
- U4 pad R7: GPIO_4 -> GPIO_3
- U4 pad T10: unconnected-(U4I-TCK-PadT10) -> TCK
- U4 pad T11: unconnected-(U4I-TMS-PadT11) -> TMS
- U4 pad T13: unconnected-(U4E-PR65B/-/HS/RDQSN65-PadT13) -> D1_5
- U4 pad T14: D1_23 -> D1_9
- U4 pad T15: D1_19 -> D1_13
- U4 pad T6: unconnected-(U4H-PB4A/+/D7/IO7-PadT6) -> GPIO_0
Routing:
- net D1_30: track 0.00 -> 32.5 mm, vias 0 -> 2
- net D1_28: track 0.00 -> 30.3 mm, vias 0 -> 2
- net D0_31: track 0.00 -> 29.1 mm, vias 0 -> 2
- net D0_29: track 0.00 -> 27.5 mm, vias 0 -> 2
- net CLK_SPI_MISO: track 26.8 -> 0.00 mm, vias 2 -> 0
- net D1_31: track 0.00 -> 26.5 mm
- net D0_30: track 0.00 -> 26.2 mm
- net CLK_SPI_MOSI: track 25.8 -> 0.00 mm, vias 2 -> 0
- net CLK_SPI_CS: track 25.0 -> 0.00 mm, vias 2 -> 0
- net D0_28: track 0.00 -> 24.6 mm
- net D1_29: track 0.00 -> 24.3 mm
- net CLK_SPI_CLK: track 24.0 -> 0.00 mm, vias 2 -> 0
- net D1_26: track 5.33 -> 29.3 mm, vias 1 -> 2
- net D0_27: track 2.97 -> 26.7 mm, vias 0 -> 2
- net D0_25: track 2.97 -> 25.1 mm, vias 0 -> 2
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Other:
- board size 50 x 35 mm -> 52 x 52 mm
- copper layers 4 -> 6
- board text added: "50 MHz"
- board text removed: "Si5340"
