File: usb-base.kicad_sch (KiCad schematic)
At the start: 28 parts, among them J1 USB3_B, J2 USB_C_Receptacle, U1 CYUSB3082-FCAXI, U2 TPS25221, U3 TPS62161DSG, U4 LFE5U-25F-6BG256C, U5 TPS62160DSG, U6 TPS62162DSG, Y1 24MHz, Y2 25MHz

Commit message: lots of work on layout
Parts:
- removed J1: USB3_B, Infineon:SAMTEC_USB3-B-S-F-TH, symbol Connector:USB3_B
- removed Y2: 25MHz, Crystal:Crystal_SMD_SeikoEpson_TSX3225-4Pin_3.2x2.5mm, symbol Oscillator:SG-5032CBN
- added C12, C13: 100n, Capacitor_SMD:C_0402_1005Metric, symbol Device:C_Small
- added C14: 10u, Capacitor_SMD:C_0805_2012Metric, symbol Device:C_Small
- added C15: 22u, Capacitor_SMD:C_1206_3216Metric, symbol Device:C_Small
- added L4: 2.2u, Inductor_SMD:L_Sunlord_SWPA3015S, symbol Device:L_Small
- added R6, R7, R8, R9: R, Resistor_SMD:R_0402_1005Metric, symbol Device:R_Small
- added U7: Si5340, Package_DFN_QFN:QFN-44-1EP_7x7mm_P0.5mm_EP5.2x5.2mm, symbol Si5340:Si5340
- added U8: TPS62160DSG, Package_SON:WSON-8-1EP_2x2mm_P0.5mm_EP0.9x1.6mm_ThermalVias, symbol Regulator_Switching:TPS62160DSG
- added Y2: 48MHz, symbol Device:Crystal_GND24
- C7, C8: footprint (none) -> Capacitor_SMD:C_0402_1005Metric
- J2: footprint (none) -> Connector_USB:USB_C_Receptacle_Amphenol_12401548E4-2A
- R4, R5: footprint (none) -> Resistor_SMD:R_0402_1005Metric
- U1: footprint Infineon:BGA169N075P13X13_10X10X120 -> library:BGA169N075P13X13_10X10X120
Connections:
- net +3V3 is gone; now on net +3.3V: U1.A3 (V33), U1.C11 (VDDIO_QSPI), U1.C3 (VDDIO_P0), U1.C5 (VDDIO_P1), U1.C7 (VDDIO_P1_CTRL), U1.C9 (VDDIO_P1), U1.E3 (VDDIO_P0_CTRL), U1.F7 (VDDIO), U1.G3 (VDDIO_P0), U1.J3 (V33), U1.L10 (V33), U1.L13 (VDDIO), U1.M12 (VDDIO_XTAL), U4.F10 (VCCIO1[2]), U4.F11 (VCCIO1[2]), U4.F6 (VCCIO0[2]), U4.F7 (VCCIO0[2]), U4.H11 (VCCIO2[2]), U4.H6 (VCCIO7[2]), U4.H7 (VCCIO7[2]), U4.J11 (VCCIO2[2]), U4.J6 (VCCIO6[2]), U4.J7 (VCCIO6[2]), U4.K11 (VCCIO3[2]), U4.L11 (VCCIO3[2]), U4.L6 (VCCIO8), U4.N10 (CFG_0)
- net USBSS_RX+ is gone; now on net USBSS_RX1+: U1.M3 (USB3RX1_P)
- net USBSS_RX- is gone; now on net USBSS_RX1-: U1.N3 (USB3RX1_N)
- net +3.3V: now also U7.18 (VDDO0), U7.23 (VDDO1), U7.26 (VDDS), U7.29 (VDDO2), U7.34 (VDDO3), U7.8 (VDDA), U7.9 (VDDA)
- net +5V: now also C14.1, U8.2 (VIN), U8.3 (EN)
- net GND: now also J2.A1 (GND), J2.A12 (GND), J2.B1 (GND), J2.B12 (GND), J2.SH (SHIELD), C14.2, C15.2, R7.2, R8.1, R9.1, U7.45 (GND), U8.1 (PGND), U8.4 (AGND), U8.9 (PAD)
- net USBHS_D+: now also J2.A6 (D+), J2.B6 (D+)
- net USBHS_D-: now also J2.A7 (D-), J2.B7 (D-)
- net VBUS_IN: now also J2.A4 (VBUS), J2.A9 (VBUS), J2.B4 (VBUS), J2.B9 (VBUS)
- net USBSS_RX2+: now reaches U1.M7 (USB3TX2_P)
- net USBSS_RX2+: now also J2.A11 (RX2+)
- net USBSS_TX2+: now reaches U1.M9 (USB3RX2_P)
- net USBSS_TX2+: now also C13.2
- net USBSS_RX2-: now reaches U1.N7 (USB3TX2_N)
- net USBSS_RX2-: now also J2.A10 (RX2-)
- net USBSS_TX2-: now reaches U1.N9 (USB3RX2_N)
- net USBSS_TX2-: now also C12.2
- net CLK2: now reaches U4.C8 (PT44A/+/PCLKT1_0)
- net CLK2: now also U7.24 (OUT1b)
- net CLK1: now reaches U4.E8 (PT42A/+/PCLKT1_1)
- net CLK1: now also U7.30 (OUT2b)
- net TX1-: now reaches C7.1
- net TX1-: now also J2.A3 (TX1-)
- net TX1+: now reaches J2.A2 (TX1+)
- net TX1+: now also C8.1
- net at J2.A5 (CC1): now also R9.2
- net USBSS_RX1-: now reaches J2.B10 (RX1-)
- net USBSS_RX1+: now reaches J2.B11 (RX1+)
- net TX2+: now reaches J2.B2 (TX2+)
- net TX2+: now also C13.1
- net TX2-: now reaches J2.B3 (TX2-)
- net TX2-: now also C12.1
- net at J2.B5 (CC2): now also R8.2
- net CLK_SPI_MOSI: now reaches U1.E5 (P7_2_SPIDAT2)
- net CLK_SPI_MOSI: now also U7.13 (SDA/SDIO)
- net CLK_SPI_MISO: now reaches U1.E6 (P7_3_SPIDAT3)
- net CLK_SPI_MISO: now also U7.15 (A1/SDO)
- net CLK_SPI_CLK: now reaches U1.F5 (P7_0_SPIDAT0)
- net CLK_SPI_CLK: now also U7.14 (SCLK)
- net CLK_SPI_CS: now reaches U1.F6 (P7_1_SPIDAT1)
- net CLK_SPI_CS: now also U7.16 (A0/CSb)
- net +1V8 renamed +1.8V
- net +1.8V: now also U7.21 (VDD), U7.32 (VDD), U7.39 (VDD), U7.40 (VDD)
- net +2V5 renamed +2.5V
- net 24MHz renamed 24MHZ
- net 25MHz renamed 100MHZ
- net 100MHZ: now also U7.20 (OUT0)
- net USBSS_TX+ renamed USBSS_TX1+
- net USBSS_TX- renamed USBSS_TX1-
- new net: U7.5 (XA), Y2.1
- new net: U7.4 (X1), U7.7 (X2), Y2.2 (G), Y2.4 (G)
- new net: U7.6 (XB), Y2.3
- new net: R6.2, R7.1, U8.5 (FB)
- new net: L4.1, U8.7 (SW)
- new net 10MHZ_IN: U7.43 (IN0)
- new net 10MHZ_OUT: U7.36 (OUT3)
- new net 2.5V: C15.1, L4.2, R6.1, U8.6 (VOS)
- new net CLK1_OUT: U7.31 (OUT2)
- new net CLK2_OUT: U7.25 (OUT1)
- no-connect marks 86 -> 87
Other:
- note added: "2.5V buck converter (FPGA VCCAUX)"
- note removed: "2.5V linear regularor (FPGA VCCAUX)"
- moved on the sheet: C4, C7, C8, J2, U1A

Commit message: Lots of routing for connectors
Parts:
- removed U7: Si5340, Package_DFN_QFN:QFN-44-1EP_7x7mm_P0.5mm_EP5.2x5.2mm, symbol Si5340:Si5340
- removed Y2: 48MHz, symbol Device:Crystal_GND24
- added C16, C18, C20, C22, C24, C26, C28, C30, C32, C34, C36, C38, C40, C42, C44, C46, C48, C50, C52, C54, C56, C58, C60: 10n, symbol Device:C_Small
- added C17, C19, C21, C23, C25, C27, C29, C31, C33, C35, C37, C39, C41, C43, C45, C47, C49, C51, C53, C55, C57, C59, C61: 100n, symbol Device:C_Small
- added J1, J2: Conn_02x35_Odd_Even, Connector_Hirose_DF40:Hirose_DF40C-70DS-0.4V_2x35_P0.4mm, symbol Connector_Generic:Conn_02x35_Odd_Even
- added R10, R3: 10k, symbol Device:R_Small
- added SW1, SW2: SW_Push, symbol Switch:SW_Push
- added Y2: 50MHz, Crystal:Crystal_SMD_SeikoEpson_TSX3225-4Pin_3.2x2.5mm, symbol Oscillator:SG-5032CBN
- J3: renamed from J2; footprint Connector_USB:USB_C_Receptacle_Amphenol_12401548E4-2A -> Connector_USB:USB_C_Receptacle_Amphenol_12401610E4-2A
Connections:
- net +1.8V: now also C16.1, C17.1, C18.1, C19.1, C20.1, C21.1, C22.1, C23.1, C24.1, C25.1, C26.1, C27.1, C28.1, C29.1, C36.1, C37.1, C38.1, C39.1, C40.1, C41.1, R3.1
- net +3.3V: now also C30.1, C31.1, C32.1, C33.1, C34.1, C35.1, C42.1, C43.1, C44.1, C45.1, C46.1, C47.1, C48.1, C49.1, C50.1, C51.1, C52.1, C53.1, C54.1, C55.1, C56.1, C57.1, C58.1, C59.1, C60.1, C61.1, J1.1 (Pin_1), J1.2 (Pin_2), J1.4 (Pin_4), J1.69 (Pin_69), J2.1 (Pin_1), J2.2 (Pin_2), J2.4 (Pin_4), SW2.2, Y2.1 (~{ST}), Y2.4 (VCC)
- net D0_0: now also U4.F12 (PR17D/-/RDQ17), J1.5 (Pin_5); no longer U4.B16 (PR11A/+/URC_GPLL0T_IN/HS/RDQ17)
- net D0_1: now also U4.H12 (PR26A/+/HS/RDQ29), J1.8 (Pin_8); no longer U4.B15 (PR11B/-/URC_GPLL0C_IN/HS/RDQ17)
- net D0_10: now also U4.B16 (PR11A/+/URC_GPLL0T_IN/HS/RDQ17), J1.25 (Pin_25); no longer U4.F13 (PR17C/+/RDQ17)
- net D0_11: now also U4.E14 (PR14C/+/RDQ17), J1.28 (Pin_28); no longer U4.G13 (PR20B/-/HS/RDQ17)
- net D0_12: now also U4.C15 (PR14B/-/HS/RDQ17), J1.29 (Pin_29); no longer U4.F15 (PR20C/+/RDQ17)
- net D0_13: now also U4.H13 (PR26B/-/HS/RDQ29), J1.32 (Pin_32); no longer U4.E16 (PR20D/-/RDQ17)
- net D0_14: now also U4.C16 (PR14A/+/HS/RDQ17), J1.33 (Pin_33); no longer U4.F16 (PR23A/+/HS/RDQ29)
- net D0_15: now also U4.F14 (PR14D/-/RDQ17), J1.36 (Pin_36); no longer U4.G15 (PR23B/-/HS/RDQ29)
- net D0_16: now also U4.D16 (PR17A/+/HS/RDQS17), J1.37 (Pin_37); no longer U4.G14 (PR23C/+/VREF1_2/RDQ29)
- net D0_17: now also U4.G14 (PR23C/+/VREF1_2/RDQ29), J1.40 (Pin_40); no longer U4.H14 (PR23D/-/RDQ29)
- net D0_18: now also U4.E15 (PR17B/-/HS/RDQSN17), J1.41 (Pin_41); no longer U4.H13 (PR26B/-/HS/RDQ29)
- net D0_19: now also U4.H14 (PR23D/-/RDQ29), J1.44 (Pin_44); no longer U4.J13 (PR26C/+/RDQ29)
- net D0_2: now also U4.F13 (PR17C/+/RDQ17), J1.9 (Pin_9); no longer U4.C14 (PR11C/+/RDQ17)
- net D0_20: now also U4.E16 (PR20D/-/RDQ17), J1.45 (Pin_45); no longer U4.G16 (PR29A/+/GR_PCLK2_1/HS/RDQS29)
- net D0_21: now also U4.J14 (PR29C/+/GR_PCLK2_0/RDQ29), J1.48 (Pin_48); no longer U4.H15 (PR29B/-/HS/RDQSN29)
- net D0_22: now also U4.F15 (PR20C/+/RDQ17), J1.49 (Pin_49); no longer U4.J14 (PR29C/+/GR_PCLK2_0/RDQ29)
- net D0_23: now also J1.52 (Pin_52)
- net D0_24: now also U4.F16 (PR23A/+/HS/RDQ29), J1.53 (Pin_53); no longer U4.J16 (PR32A/+/PCLKT2_1/HS/RDQ29)
- net D0_25: now also U4.G15 (PR23B/-/HS/RDQ29), J1.56 (Pin_56); no longer U4.J15 (PR32B/-/PCLKC2_1/HS/RDQ29)
- net D0_26: now also U4.G16 (PR29A/+/GR_PCLK2_1/HS/RDQS29), J1.57 (Pin_57); no longer U4.K16 (PR32C/+/PCLKT2_0/RDQ29)
- net D0_27: now also U4.H15 (PR29B/-/HS/RDQSN29), J1.60 (Pin_60); no longer U4.K15 (PR32D/-/PCLKC2_0/RDQ29)
- net D0_3: now also U4.G12 (PR20A/+/HS/RDQ17), J1.12 (Pin_12); no longer U4.D14 (PR11D/-/RDQ17)
- net D0_4: now also U4.C14 (PR11C/+/RDQ17), J1.13 (Pin_13); no longer U4.C16 (PR14A/+/HS/RDQ17)
- net D0_5: now also U4.J12 (PR26D/-/RDQ29), J1.16 (Pin_16); no longer U4.C15 (PR14B/-/HS/RDQ17)
- net D0_6: now also U4.D14 (PR11D/-/RDQ17), J1.17 (Pin_17); no longer U4.E14 (PR14C/+/RDQ17)
- net D0_7: now also U4.G13 (PR20B/-/HS/RDQ17), J1.20 (Pin_20); no longer U4.F14 (PR14D/-/RDQ17)
- net D0_8: now also U4.B15 (PR11B/-/URC_GPLL0C_IN/HS/RDQ17), J1.21 (Pin_21); no longer U4.D16 (PR17A/+/HS/RDQS17)
- net D0_9: now also U4.J13 (PR26C/+/RDQ29), J1.24 (Pin_24); no longer U4.E15 (PR17B/-/HS/RDQSN17)
- net D1_0: now also U4.N11 (PR68B/-/HS/RDQ65), J2.5 (Pin_5); no longer U4.L16 (PR35A/+/PCLKT3_1/HS/RDQ41)
- net D1_1: now also U4.P11 (PR68C/+/LRC_GPLL0T_IN/RDQ65), J2.8 (Pin_8); no longer U4.L15 (PR35B/-/PCLKC3_1/HS/RDQ41)
- net D1_10: now also U4.N12 (PR65D/-/RDQ65), J2.25 (Pin_25); no longer U4.L14 (PR41C/+/RDQ41)
- net D1_11: now also U4.R14 (PR62B/-/HS/RDQ65), J2.28 (Pin_28); no longer U4.M14 (PR41D/-/RDQ41)
- net D1_12: now also U4.P13 (PR62A/+/HS/RDQ65), J2.29 (Pin_29); no longer U4.P16 (PR44A/+/HS/RDQ41)
- net D1_13: now also U4.T15 (PR59D/-/RDQ65), J2.32 (Pin_32); no longer U4.R16 (PR44B/-/VREF1_3/HS/RDQ41)
- net D1_14: now also U4.N13 (PR59A/+/HS/RDQ65), J2.33 (Pin_33); no longer U4.M13 (PR44C/+/RDQ41)
- net D1_15: now also U4.R15 (PR59C/+/RDQ65), J2.36 (Pin_36); no longer U4.N14 (PR44D/-/RDQ41)
- net D1_16: now also U4.P14 (PR59B/-/HS/RDQ65), J2.37 (Pin_37); no longer U4.N13 (PR59A/+/HS/RDQ65)
- net D1_17: now also U4.R16 (PR44B/-/VREF1_3/HS/RDQ41), J2.40 (Pin_40); no longer U4.P14 (PR59B/-/HS/RDQ65)
- net D1_18: now also U4.N14 (PR44D/-/RDQ41), J2.41 (Pin_41); no longer U4.R15 (PR59C/+/RDQ65)
- net D1_19: now also U4.P15 (PR41B/-/HS/RDQSN41), J2.44 (Pin_44); no longer U4.T15 (PR59D/-/RDQ65)
- net D1_2: now also U4.M11 (PR68A/+/HS/RDQ65), J2.9 (Pin_9); no longer U4.M16 (PR35C/+/PCLKT3_0/RDQ41)
- net D1_20: now also U4.M13 (PR44C/+/RDQ41), J2.45 (Pin_45); no longer U4.P13 (PR62A/+/HS/RDQ65)
- net D1_21: now also U4.P16 (PR44A/+/HS/RDQ41), J2.48 (Pin_48); no longer U4.R14 (PR62B/-/HS/RDQ65)
- net D1_22: now also U4.M14 (PR41D/-/RDQ41), J2.49 (Pin_49); no longer U4.R13 (PR62C/+/RDQ65)
- net D1_23: now also U4.N16 (PR41A/+/HS/RDQS41), J2.52 (Pin_52); no longer U4.T14 (PR62D/-/RDQ65)
- net D1_24: now also U4.L14 (PR41C/+/RDQ41), J2.53 (Pin_53); no longer U4.R12 (PR65A/+/HS/RDQS65)
- net D1_25: now also U4.M16 (PR35C/+/PCLKT3_0/RDQ41), J2.56 (Pin_56); no longer U4.M12 (PR65C/+/RDQ65)
- net D1_26: now also U4.L13 (PR38C/+/GR_PCLK3_1/RDQ41), J2.57 (Pin_57); no longer U4.N12 (PR65D/-/RDQ65)
- net D1_27: now also U4.M15 (PR35D/-/PCLKC3_0/RDQ41), J2.60 (Pin_60); no longer U4.P12 (PR68D/-/LRC_GPLL0C_IN/RDQ65)
- net D1_3: now also U4.R12 (PR65A/+/HS/RDQS65), J2.12 (Pin_12); no longer U4.M15 (PR35D/-/PCLKC3_0/RDQ41)
- net D1_4: now also U4.M12 (PR65C/+/RDQ65), J2.13 (Pin_13); no longer U4.K13 (PR38A/+/GR_PCLK3_0/HS/RDQ41)
- net D1_5: now also U4.T13 (PR65B/-/HS/RDQSN65), J2.16 (Pin_16); no longer U4.K12 (PR38B/-/HS/RDQ41)
- net D1_6: now also U4.L12 (PR38D/-/RDQ41), J2.17 (Pin_17); no longer U4.L13 (PR38C/+/GR_PCLK3_1/RDQ41)
- net D1_7: now also U4.R13 (PR62C/+/RDQ65), J2.20 (Pin_20); no longer U4.L12 (PR38D/-/RDQ41)
- net D1_8: now also U4.P12 (PR68D/-/LRC_GPLL0C_IN/RDQ65), J2.21 (Pin_21); no longer U4.N16 (PR41A/+/HS/RDQS41)
- net D1_9: now also U4.T14 (PR62D/-/RDQ65), J2.24 (Pin_24); no longer U4.P15 (PR41B/-/HS/RDQSN41)
- net DONE: now also U1.J12 (P9_7_I2S0-RXMCLK); no longer U1.H13 (P0_0_P0SDA)
- net GND: now also C16.2, C17.2, C18.2, C19.2, C20.2, C21.2, C22.2, C23.2, C24.2, C25.2, C26.2, C27.2, C28.2, C29.2, C30.2, C31.2, C32.2, C33.2, C34.2, C35.2, C36.2, C37.2, C38.2, C39.2, C40.2, C41.2, C42.2, C43.2, C44.2, C45.2, C46.2, C47.2, C48.2, C49.2, C50.2, C51.2, C52.2, C53.2, C54.2, C55.2, C56.2, C57.2, C58.2, C59.2, C60.2, C61.2, J1.10 (Pin_10), J1.11 (Pin_11), J1.14 (Pin_14), J1.15 (Pin_15), J1.18 (Pin_18), J1.19 (Pin_19), J1.22 (Pin_22), J1.23 (Pin_23), J1.26 (Pin_26), J1.27 (Pin_27), J1.3 (Pin_3), J1.30 (Pin_30), J1.31 (Pin_31), J1.34 (Pin_34), J1.35 (Pin_35), J1.38 (Pin_38), J1.39 (Pin_39), J1.42 (Pin_42), J1.43 (Pin_43), J1.46 (Pin_46), J1.47 (Pin_47), J1.50 (Pin_50), J1.51 (Pin_51), J1.54 (Pin_54), J1.55 (Pin_55), J1.58 (Pin_58), J1.59 (Pin_59), J1.6 (Pin_6), J1.62 (Pin_62), J1.63 (Pin_63), J1.66 (Pin_66), J1.67 (Pin_67), J1.7 (Pin_7), J1.70 (Pin_70), J2.10 (Pin_10), J2.11 (Pin_11), J2.14 (Pin_14), J2.15 (Pin_15), J2.18 (Pin_18), J2.19 (Pin_19), J2.22 (Pin_22), J2.23 (Pin_23), J2.26 (Pin_26), J2.27 (Pin_27), J2.3 (Pin_3), J2.30 (Pin_30), J2.31 (Pin_31), J2.34 (Pin_34), J2.35 (Pin_35), J2.38 (Pin_38), J2.39 (Pin_39), J2.42 (Pin_42), J2.43 (Pin_43), J2.46 (Pin_46), J2.47 (Pin_47), J2.50 (Pin_50), J2.51 (Pin_51), J2.54 (Pin_54), J2.55 (Pin_55), J2.58 (Pin_58), J2.59 (Pin_59), J2.6 (Pin_6), J2.62 (Pin_62), J2.63 (Pin_63), J2.66 (Pin_66), J2.67 (Pin_67), J2.69 (Pin_69), J2.7 (Pin_7), J2.70 (Pin_70), R10.2, SW1.1, Y2.2 (GND)
- net GPIO_0: now also U4.T6 (PB4A/+/D7/IO7); no longer U4.R6 (PB4B/-/D6/IO6)
- net GPIO_1: now also U1.H13 (P0_0_P0SDA); no longer U1.J12 (P9_7_I2S0-RXMCLK)
- net GPIO_2: now also U4.M7 (PB9B/-/D2/IO2); no longer U4.N7 (PB9A/+/D3/IO3)
- net GPIO_3: now also U4.R7 (PB6A/+/D5/MISO2/IO5); no longer U4.P7 (PB6B/-/D4/MOSI2/IO4)
- net GPIO_4: now also U4.P7 (PB6B/-/D4/MOSI2/IO4); no longer U4.R7 (PB6A/+/D5/MISO2/IO5)
- net GPIO_5: now also U4.R6 (PB4B/-/D6/IO6); no longer U4.M7 (PB9B/-/D2/IO2)
- net PMODE: now also R10.1, SW2.1
- net RESET: now reaches U1.K6 (XRES_N)
- net RESET: now also R3.2, SW1.2
- net TDO: now reaches U4.M10 (TDO)
- net TDI: now reaches U4.R11 (TDI)
- net TCK: now reaches U4.T10 (TCK)
- net TMS: now reaches U4.T11 (TMS)
- net 100MHZ renamed 50MHz
- net 50MHz: now also Y2.3 (OUT)
- net CLK1: no longer names the net of U4.E8 (PT42A/+/PCLKT1_1)
- net CLK2: no longer names the net of U4.C8 (PT44A/+/PCLKT1_0)
- new net D0_28: J1.61 (Pin_61), U4.J15 (PR32B/-/PCLKC2_1/HS/RDQ29)
- new net D0_29: J1.64 (Pin_64), U4.J16 (PR32A/+/PCLKT2_1/HS/RDQ29)
- new net D0_30: J1.65 (Pin_65), U4.K15 (PR32D/-/PCLKC2_0/RDQ29)
- new net D0_31: J1.68 (Pin_68), U4.K16 (PR32C/+/PCLKT2_0/RDQ29)
- new net D1_28: J2.61 (Pin_61), U4.K13 (PR38A/+/GR_PCLK3_0/HS/RDQ41)
- new net D1_29: J2.64 (Pin_64), U4.L16 (PR35A/+/PCLKT3_1/HS/RDQ41)
- new net D1_30: J2.65 (Pin_65), U4.K12 (PR38B/-/HS/RDQ41)
- new net D1_31: J2.68 (Pin_68), U4.L15 (PR35B/-/PCLKC3_1/HS/RDQ41)
- no-connect marks 87 -> 75
Other:
- note added: "FX5 Power"
- note added: "TODO: ESD Protection"
- note added: "USB3V18"
- note added: "V33"
- note added: "VDDD"
- note added: "VDDIO"
- note added: "VDDIOQSPI VDDIOXTAL"
- note added: "VDDIO_P0"
- note added: "VDDIO_P1"
- note removed: "FX5 Power TODO: Decoupling"
- moved on the sheet: C12, C13, C4, C7, C8, J3, R8, R9, U1A
